File: 2choc2flat-extmcu.kicad_sch (KiCad schematic)
At the start: 175 parts, among them J1 HRO-TYPE-C-31-M-12, J2 ISP, J3 ai03_ud, K1 KEYSW, K10 KEYSW, K11 KEYSW, K12 KEYSW, K13 KEYSW, K14 KEYSW, K15 KEYSW, K15-1 KEYSW, K16 KEYSW, K17 KEYSW, K18 KEYSW, K19 KEYSW, K2 KEYSW, K20 KEYSW, K21 KEYSW, K22 KEYSW, K23 KEYSW, K24 KEYSW, K25 KEYSW, K26 KEYSW, K27 KEYSW, K28 KEYSW, K29 KEYSW, K3 KEYSW, K31 KEYSW, K31-1 KEYSW, K32 KEYSW, K33 KEYSW, K34 KEYSW, K35 KEYSW, K36 KEYSW, K37 KEYSW, K38 KEYSW, K39 KEYSW, K4 KEYSW, K40 KEYSW, K41 KEYSW, K42 KEYSW, K43 KEYSW, K44 KEYSW, K44-1 KEYSW, K46 KEYSW, K46-1 KEYSW, K47 KEYSW, K48 KEYSW, K49 KEYSW, K5 KEYSW, K50 KEYSW, K51 KEYSW, K52 KEYSW, K53 KEYSW, K54 KEYSW, K55 KEYSW, K56 KEYSW, K57 KEYSW, K58 KEYSW, K58-1 KEYSW, K59 KEYSW, K6 KEYSW, K61 KEYSW, K61-1 KEYSW, K62 KEYSW, K62-1 KEYSW, K63 KEYSW, K63-1 KEYSW, K67 KEYSW, K67-1 KEYSW, K7 KEYSW, K71 KEYSW, K72 KEYSW, K72-1 KEYSW, K73 KEYSW, K73-1 KEYSW, K74 KEYSW, K74-1 KEYSW, K8 KEYSW, K9 KEYSW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

Commit message: lshift stab support
Parts:
- removed C1: 1u, Keeb_components:C_0805, symbol Device:C
- removed C2, C3, C4, C5: 0.1u, Keeb_components:C_0805, symbol Device:C
- removed C6: 4.7u, Keeb_components:C_0805, symbol Device:C
- removed D47: D, Keeb_components:D_0805, symbol Device:D
- removed F1: Polyfuse, Keeb_components:R_0805, symbol Device:Polyfuse
- removed H1: B0, footprints:free_pin, symbol Connector_Generic:Conn_01x01
- removed H3: GND, footprints:free_pin, symbol Connector_Generic:Conn_01x01
- removed H4: +5v, footprints:free_pin, symbol Connector_Generic:Conn_01x01
- removed J1: HRO-TYPE-C-31-M-12, Keeb_components:HRO-TYPE-C-31-M-12, symbol Type-C:HRO-TYPE-C-31-M-12
- removed J2: ISP, Keeb_components:isp_standard, symbol Connector_Generic:Conn_02x03_Odd_Even
- removed J3: ai03_ud, Keeb_components:JST_SH_SM04B-SRSS-TB_1x04-1MP_P1.00mm_Horizontal, symbol Connector_Generic:Conn_01x04
- removed K15: KEYSW, Keeb_switches:CHERRY_PCB_200H, symbol keyboard_parts:KEYSW
- removed K46-1: KEYSW, Keeb_switches:CHERRY_PLATE_125H, symbol keyboard_parts:KEYSW
- removed K47, K62-1, K73-1: KEYSW, Keeb_switches:CHERRY_PLATE_100H, symbol keyboard_parts:KEYSW
- removed K58: KEYSW, Keeb_switches:CHERRY_PCB_275H, symbol keyboard_parts:KEYSW
- removed K61-1, K63-1, K72-1, K74-1: KEYSW, Keeb_switches:CHERRY_PLATE_150H, symbol keyboard_parts:KEYSW
- removed K67-1: KEYSW, Keeb_switches:CHERRY_PCB_700H_F, symbol keyboard_parts:KEYSW
- removed LS1: Speaker, Keeb_components:speaker_AST1109MLTRQ, symbol Device:Speaker
- removed R1, R2: 22, Keeb_components:R_0805, symbol Device:R
- removed R3, R4: 5.1k, Keeb_components:R_0805, symbol Device:R
- removed R5, R6: 10k, Keeb_components:R_0805, symbol Device:R
- removed S7, S8, S9: Tofu screw, footprints:5.5_5x2.5mm, symbol Connector:Screw_Terminal_01x01
- removed SW1: SW_PUSH, Button_Switch_SMD:SW_SPST_TL3342, symbol keyboard_parts:SW_PUSH
- removed U1: ATmega32U4, Keeb_components:ATMEGA32U4, symbol atmel:ATmega32U4
- removed U2: USBLC6-2SC6, Keeb_components:USBLC6-2SC6, symbol keyboard_parts:USBLC6-2SC6
- removed X1: XTAL_GND, Keeb_components:Resonator_SMD_muRata_CSTNExxV-3Pin-p1.2, symbol keyboard_parts:XTAL_GND
- added J1, J3: Conn_01x09_Male, Connector_PinHeader_2.54mm:PinHeader_1x09_P2.54mm_Vertical, symbol Connector:Conn_01x09_Male
- added J2: Conn_01x05_Male, Connector_PinHeader_2.54mm:PinHeader_1x05_P2.54mm_Vertical, symbol Connector:Conn_01x05_Male
- D1, D10, D11, D12, D13, D14, D15, D16, D17, D18, D19, D2, D20, D21, D22, D23, D24, D25, D26, D27, D28, D29, D3, D31, D32, D33, D34, D35, D36, D37, D38, D39, D4, D40, D41, D42, D43, D44, D46, D48, D49, D5, D50, D51, D52, D53, D54, D55, D56, D57, D58, D59, D6, D61, D62, D63, D67, D7, D71, D72, D73, D74, D8, D9: footprint Keeb_components:D_0805 -> Diode_SMD:D_0805_2012Metric
- K1, K10, K11, K12, K13, K14, K15-1, K17, K18, K19, K2, K20, K21, K22, K23, K24, K25, K26, K27, K28, K3, K32, K33, K34, K35, K36, K37, K38, K39, K4, K40, K41, K42, K43, K48, K49, K5, K50, K51, K52, K53, K54, K55, K56, K57, K59, K6, K7, K9: footprint Keeb_switches:CHERRY_PLATE_100H -> Switch_Keyboard_Hotswap_Kailh_mine:SW_Hotswap_Kailh_Choc_V2_1.00u
- K16, K29: footprint Keeb_switches:CHERRY_PLATE_150H -> Switch_Keyboard_Hotswap_Kailh_mine:SW_Hotswap_Kailh_Choc_V2_1.50u
- K31, K58-1: footprint Keeb_switches:CHERRY_PLATE_175H -> Switch_Keyboard_Hotswap_Kailh_mine:SW_Hotswap_Kailh_Choc_V2_1.75u
- K31-1, K61, K62, K63, K71, K72, K73, K74: footprint Keeb_switches:CHERRY_PLATE_125H -> Switch_Keyboard_Hotswap_Kailh_mine:SW_Hotswap_Kailh_Choc_V2_1.25u
- K44: footprint Keeb_switches:CHERRY_PCB_225H -> Switch_Keyboard_Hotswap_Kailh_mine:SW_Hotswap_Kailh_Choc_V2_2.25u
- K44-1: footprint Keeb_switches:CHERRY_PCB_200H_V -> Switch_Keyboard_Hotswap_Kailh_mine:SW_Hotswap_Kailh_Choc_V2_ISOEnter_270deg
- K46: footprint Keeb_switches:CHERRY_PCB_225H -> Switch_Keyboard_Kailh_mine:SW_Kailh_Choc_V2_2.25u_Gateron_LP_Stabs
- K67: footprint Keeb_switches:CHERRY_PCB_625H_F -> Switch_Keyboard_Hotswap_Kailh_mine:SW_Hotswap_Kailh_Choc_V2_6.25u
- K8: footprint Keeb_switches:CHERRY_PLATE_100H -> Switch_Keyboard_Kailh_mine:SW_Kailh_Choc_V2_1.00u
- S3: footprint footprints:5.5_5x2.5mm -> MountingHole:MountingHole_2.2mm_M2_Pad_TopOnly
Connections:
- net GND: now also J1.2 (Pin_2)
- net col0: now also K1.1, K16.2, K31-1.1, J1.4 (Pin_4); no longer K1.2, K16.1, K31-1.2
- net col1: now also J1.5 (Pin_5)
- net col10: now also J3.5 (Pin_5)
- net col11: now also J3.4 (Pin_4)
- net col12: now also J3.3 (Pin_3)
- net col13: now also K29.2, J3.2 (Pin_2); no longer K29.1
- net col14: now also J3.1 (Pin_1)
- net col2: now also J1.6 (Pin_6)
- net col3: now also J1.7 (Pin_7)
- net col4: now also J1.8 (Pin_8)
- net col5: now also J1.9 (Pin_9)
- net col6: now also J2.4 (Pin_4)
- net col7: now also J2.5 (Pin_5)
- net col8: now also J3.7 (Pin_7)
- net col9: now also J3.6 (Pin_6)
- net row0: now also J2.1 (Pin_1)
- net row1: now also J2.2 (Pin_2)
- net row2: now also J2.3 (Pin_3)
- net row3: now also J3.9 (Pin_9)
- net row4: now also J3.8 (Pin_8)
- net at D1.2 (A): now also K1.2; no longer K1.1
- net at D16.2 (A): now also K16.1; no longer K16.2
- net at D29.2 (A): now also K29.1; no longer K29.2
- net at D31.2 (A), K31.1: now also K31-1.2; no longer K31-1.1
- new net +3V3: J1.3 (Pin_3)
- new net +5V: J1.1 (Pin_1)
- no-connect marks 3 -> 0
Other:
- moved on the sheet: K15-1, K58-1
