File: choc2-gateron-lp-tester/choc2-gateron-lp-tester.kicad_pcb (KiCad board)
At the start: 2 copper layers, 45.7 x 68.6 mm, 10 parts, among them SW1 SW_Push

Commit message: resize to save costs
Parts:
- moved H2 6.35 mm to (108.0, 106.7)
- moved H3 6.35 mm to (146.1, 106.7)
- moved H1 6.35 mm to (108.0, 83.8)
- moved H4 6.35 mm to (146.1, 83.8)
- moved H9 6.35 mm to (127.0, 95.2)
Other:
- board size 45.7 x 68.6 mm -> 45.7 x 62.2 mm
- board text added: "CUT OUT"
- board text added: "Gateron Low-Profile Stabs + Kailh Choc v2 Tester"
Changed lines of the file:
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@@
       (layerselection 0x00010fc_ffffffff)
       (disableapertmacros false)
-      (usegerberextensions false)
+      (usegerberextensions true)
       (usegerberattributes true)
       (usegerberadvancedattributes true)
@@
       (plotinvisibletext false)
       (sketchpadsonfab false)
-      (subtractmaskfromsilk false)
+      (subtractmaskfromsilk true)
       (outputformat 1)
       (mirror false)
-      (drillshape 1)
+      (drillshape 0)
       (scaleselection 1)
-      (outputdirectory "")
+      (outputdirectory "./gerbers")
     )
   )
@@
   )
   (footprint "MountingHole:MountingHole_2.2mm_M2" (layer "F.Cu")
-    (at 107.95 100.33)
+    (at 107.95 106.68)
     (descr "Mounting Hole 2.2mm, no annular, M2")
     (tags "mounting hole 2.2mm no annular m2")
@@
   )
   (footprint "MountingHole:MountingHole_2.2mm_M2" (layer "F.Cu")
-    (at 146.05 100.33)
+    (at 146.05 106.68)
     (descr "Mounting Hole 2.2mm, no annular, M2")
     (tags "mounting hole 2.2mm no annular m2")
@@
   )
   (footprint "MountingHole:MountingHole_2.2mm_M2" (layer "F.Cu")
-    (at 146.05 77.47 180)
+    (at 146.05 83.82 180)
     (descr "Mounting Hole 2.2mm, no annular, M2")
     (tags "mounting hole 2.2mm no annular m2")
@@
   )
   (footprint "MountingHole:MountingHole_2.2mm_M2" (layer "F.Cu")
-    (at 107.95 77.47 180)
+    (at 107.95 83.82 180)
     (descr "Mounting Hole 2.2mm, no annular, M2")
     (tags "mounting hole 2.2mm no annular m2")
@@
   )
   (footprint "Mounting_Keyboard_Stabilizer:Cherry_Plate_Stabilizer_Cutout_2.00u" (layer "F.Cu")
-    (at 127 88.9)
+    (at 127 95.25)
     (property "Sheetfile" "choc2-gateron-lp-tester.kicad_sch")
     (property "Sheetname" "")
@@
   (gr_arc (start 146.05 111.76) (mid 148.744077 112.875923) (end 149.86 115.57) (layer "Edge.Cuts") (width 0.1))
   (gr_line (start 104.14 115.57) (end 104.14 138.43) (layer "Edge.Cuts") (width 0.1))
-  (gr_line (start 104.14 77.47) (end 104.14 100.33) (layer "Edge.Cuts") (width 0.1))
+  (gr_line (start 104.14 83.82) (end 104.14 106.68) (layer "Edge.Cuts") (width 0.1))
   (gr_line (start 149.86 138.43) (end 149.86 115.57) (layer "Edge.Cuts") (width 0.1))
   (gr_arc (start 104.14 115.57) (mid 105.255923 112.875923) (end 107.95 111.76) (layer "Edge.Cuts") (width 0.1))
-  (gr_arc (start 104.14 77.47) (mid 105.255923 74.775923) (end 107.95 73.66) (layer "Edge.Cuts") (width 0.1))
-  (gr_arc (start 107.95 104.14) (mid 105.255923 103.024077) (end 104.14 100.33) (layer "Edge.Cuts") (width 0.1))
+  (gr_arc (start 104.14 83.82) (mid 105.255923 81.125923) (end 107.95 80.01) (layer "Edge.Cuts") (width 0.1))
+  (gr_arc (start 107.95 110.49) (mid 105.255923 109.374077) (end 104.14 106.68) (layer "Edge.Cuts") (width 0.1))
   (gr_arc (start 107.95 142.24) (mid 105.255923 141.124077) (end 104.14 138.43) (layer "Edge.Cuts") (width 0.1))
-  (gr_arc (start 146.05 73.66) (mid 148.744077 74.775923) (end 149.86 77.47) (layer "Edge.Cuts") (width 0.1))
+  (gr_arc (start 146.05 80.01) (mid 148.744077 81.125923) (end 149.86 83.82) (layer "Edge.Cuts") (width 0.1))
   (gr_arc (start 149.86 138.43) (mid 148.744077 141.124077) (end 146.05 142.24) (layer "Edge.Cuts") (width 0.1))
   (gr_line (start 107.95 111.76) (end 146.05 111.76) (layer "Edge.Cuts") (width 0.1))
   (gr_line (start 107.95 142.24) (end 146.05 142.24) (layer "Edge.Cuts") (width 0.1))
-  (gr_line (start 107.95 73.66) (end 146.05 73.66) (layer "Edge.Cuts") (width 0.1))
-  (gr_line (start 107.95 104.14) (end 146.05 104.14) (layer "Edge.Cuts") (width 0.1))
-  (gr_arc (start 149.86 100.33) (mid 148.744077 103.024077) (end 146.05 104.14) (layer "Edge.Cuts") (width 0.1))
-  (gr_line (start 149.86 100.33) (end 149.86 77.47) (layer "Edge.Cuts") (width 0.1))
+  (gr_line (start 107.95 80.01) (end 146.05 80.01) (layer "Edge.Cuts") (width 0.1))
+  (gr_line (start 107.95 110.49) (end 146.05 110.49) (layer "Edge.Cuts") (width 0.1))
+  (gr_arc (start 149.86 106.68) (mid 148.744077 109.374077) (end 146.05 110.49) (layer "Edge.Cuts") (width 0.1))
+  (gr_line (start 149.86 106.68) (end 149.86 83.82) (layer "Edge.Cuts") (width 0.1))
+  (gr_text "Gateron Low-Profile Stabs\n+ Kailh Choc v2 Tester" (at 127 82.55) (layer "F.Cu")
+    (effects (font (size 1 1) (thickness 0.15)))
+  )
+  (gr_text "Gateron Low-Profile Stabs\n+ Kailh Choc v2 Tester" (at 127 114.3) (layer "F.Cu")
+    (effects (font (size 1 1) (thickness 0.15)))
+  )
+  (gr_text "Gateron Low-Profile Stabs\n+ Kailh Choc v2 Tester" (at 127 114.3) (layer "F.SilkS")
+    (effects (font (size 1 1) (thickness 0.15)))
+  )
+  (gr_text "Gateron Low-Profile Stabs\n+ Kailh Choc v2 Tester" (at 127 82.55) (layer "F.SilkS")
+    (effects (font (size 1 1) (thickness 0.15)))
+  )
+  (gr_text "CUT OUT" (at 114.3 127 90) (layer "Cmts.User")
+    (effects (font (size 1 1) (thickness 0.15)))
+  )
+  (gr_text "CUT OUT" (at 139.7 127 90) (layer "Cmts.User")
+    (effects (font (size 1 1) (thickness 0.15)))
+  )
+  (gr_text "CUT OUT" (at 127 95.25) (layer "Cmts.User")
+    (effects (font (size 1 1) (thickness 0.15)))
+  )
 )
