File: 2choc2flat-extmcu-ansi/2choc2flat-extmcu-ansi.kicad_pcb (KiCad board)
At the start: 2 copper layers, 284.7 x 94.2 mm, 140 parts, among them J1 Conn_01x09_Male, J2 Conn_01x05_Male, J3 Conn_01x09_Male, K1 KEYSW, K10 KEYSW, K11 KEYSW, K12 KEYSW, K13 KEYSW, K14 KEYSW, K16 KEYSW, K17 KEYSW, K18 KEYSW, K19 KEYSW, K2 KEYSW, K20 KEYSW, K21 KEYSW, K22 KEYSW, K23 KEYSW, K24 KEYSW, K25 KEYSW, K26 KEYSW, K27 KEYSW, K28 KEYSW, K29 KEYSW, K3 KEYSW, K31 KEYSW, K31-1 KEYSW, K32 KEYSW, K33 KEYSW, K34 KEYSW, K35 KEYSW, K36 KEYSW, K37 KEYSW, K38 KEYSW, K39 KEYSW, K4 KEYSW, K40 KEYSW, K41 KEYSW, K42 KEYSW, K44 KEYSW, K46 KEYSW, K47 KEYSW, K48 KEYSW, K49 KEYSW, K5 KEYSW, K50 KEYSW, K51 KEYSW, K52 KEYSW, K53 KEYSW, K54 KEYSW, K55 KEYSW, K56 KEYSW, K57 KEYSW, K58 KEYSW, K59 KEYSW, K6 KEYSW, K61 KEYSW, K62 KEYSW, K63 KEYSW, K67 KEYSW, K7 KEYSW, K71 KEYSW, K72 KEYSW, K73 KEYSW, K74 KEYSW, K75 KEYSW, K8 KEYSW, K9 KEYSW

Commit message: routing complete
Parts:
- S3: footprint MountingHole:MountingHole_2.2mm_M2_Pad_Via -> MountingHole:MountingHole_2.2mm_M2_Pad_TopOnly
- moved R1 16.4 mm to (4.57, 44.2), turned to -90 degrees
- moved DI1 15.6 mm to (10.2, 41.7)
Connections:
- J1 pad 2: col13 -> col8
- J1 pad 3: col12 -> col9
- J1 pad 4: col11 -> col10
- J1 pad 5: col10 -> col11
- J1 pad 6: col9 -> col12
- J1 pad 7: col8 -> col13
- J2 pad 1: row0 -> row2
- J2 pad 3: row2 -> row0
- J2 pad 4: col6 -> col7
- J2 pad 5: col7 -> col6
- J3 pad 4: col1 -> col0
- J3 pad 5: col2 -> col1
- J3 pad 6: col3 -> col2
- J3 pad 7: col4 -> col3
- J3 pad 8: col5 -> col4
- J3 pad 9: col0 -> col5
Routing:
- net col12: track 19.2 -> 320.8 mm, vias 2 -> 1
- net col13: track 132.7 -> 375.1 mm, vias 0 -> 1
- net col11: track 61.2 -> 299.0 mm, vias 6 -> 1
- net col10: track 61.2 -> 279.6 mm, vias 6 -> 1
- net col9: track 61.2 -> 260.2 mm, vias 6 -> 1
- net col8: track 42.0 -> 222.2 mm, vias 4 -> 1
- net col7: track 42.7 -> 199.4 mm, vias 4 -> 1
- net col6: track 66.0 -> 199.9 mm, vias 6 -> 1
- net col5: track 42.0 -> 153.6 mm, vias 4 -> 1
- net col4: track 42.1 -> 133.1 mm, vias 4 -> 2
- net row4: track 280.5 -> 358.4 mm, vias 0 -> 2
- net col3: track 42.0 -> 112.9 mm, vias 4 -> 2
- net col0: track 30.6 -> 88.2 mm
- net row3: track 254.7 -> 306.6 mm, vias 0 -> 16
- net row2: track 230.7 -> 279.4 mm, vias 0 -> 26
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