File: 2choc2flat-extmcu-iso/2choc2flat-extmcu-iso.kicad_pcb (KiCad board)
At the start: 2 copper layers, 284.7 x 94.2 mm, 142 parts, among them J1 Conn_01x09_Male, J2 Conn_01x05_Male, J3 Conn_01x09_Male, K1 KEYSW, K10 KEYSW, K11 KEYSW, K12 KEYSW, K13 KEYSW, K14 KEYSW, K15 KEYSW, K16 KEYSW, K17 KEYSW, K18 KEYSW, K19 KEYSW, K2 KEYSW, K20 KEYSW, K21 KEYSW, K22 KEYSW, K23 KEYSW, K24 KEYSW, K25 KEYSW, K26 KEYSW, K27 KEYSW, K28 KEYSW, K29 KEYSW, K29-1 KEYSW, K3 KEYSW, K30 KEYSW, K31 KEYSW, K32 KEYSW, K33 KEYSW, K34 KEYSW, K35 KEYSW, K38 KEYSW, K39 KEYSW, K4 KEYSW, K40 KEYSW, K41 KEYSW, K42 KEYSW, K43 KEYSW, K44 KEYSW, K46 KEYSW, K47 KEYSW, K48 KEYSW, K49 KEYSW, K5 KEYSW, K50 KEYSW, K51 KEYSW, K52 KEYSW, K53 KEYSW, K54 KEYSW, K55 KEYSW, K56 KEYSW, K57 KEYSW, K58 KEYSW, K59 KEYSW, K6 KEYSW, K61 KEYSW, K62 KEYSW, K63 KEYSW, K67 KEYSW, K7 KEYSW, K71 KEYSW, K72 KEYSW, K73 KEYSW, K74 KEYSW, K75 KEYSW, K8 KEYSW, K9 KEYSW

Commit message: wip renaming stuff
Parts:
- renumbered D32 to D30, D33 to D31, D34 to D32, D35 to D33, D36 to D34, D37 to D35, D38 to D36, D39 to D37, D40 to D38, D41 to D39, D42 to D40, D43 to D41, D44 to D42, K38 to K36, K39 to K37, K40 to K38, K41 to K39, K42 to K40, K43 to K41, K44 to K42

Commit message: rerouted, capslock light
Parts:
- renumbered D46 to D43, D47 to D44, D48 to D45, D49 to D46, D50 to D47, D51 to D48, D52 to D49, D53 to D50, D54 to D51, D55 to D52, D56 to D53, D57 to D54, D58 to D55, D59 to D56, D61 to D57, D62 to D58, D63 to D59, D67 to D60, D71 to D61, D72 to D62, D73 to D63, D74 to D64, D75 to D65, K46 to K43, K47 to K44, K48 to K45, K49 to K46, K50 to K47, K51 to K48, K52 to K49, K53 to K50, K54 to K51, K55 to K52, K56 to K53, K57 to K54, K58 to K55, K59 to K56, K61 to K57, K62 to K58, K63 to K59, K67 to K60, K71 to K61, K72 to K62, K73 to K63, K74 to K64, K75 to K65
Routing:
- net Net-(D34-Pad2): track 11.0 -> 12.2 mm

Commit message: rev 1.3 layouts
Routing:
- net row0: track 307.4 -> 332.8 mm, vias 24 -> 13
- net row2: track 269.8 -> 285.3 mm, vias 23 -> 13
- net row1: track 290.7 -> 302.4 mm, vias 24 -> 15
- net row3: track 304.5 -> 309.8 mm, vias 12 -> 9
- net col13: track 370.8 -> 373.0 mm
- net col12: track 296.8 -> 298.0 mm
- net col5: track 131.7 -> 132.8 mm
- net col11: track 274.8 -> 275.7 mm
- net col10: track 252.9 -> 253.6 mm
Other:
- board text added: "2choc2flat ISO(ish) v1.3 by schizobovine <sean@yak.net>"
- board text removed: "2choc2flat ISO(ish) v1.2 by schizobovine <sean@yak.net>"
