File: 2choc2flat-extmcu-iso/2choc2flat-extmcu-iso.kicad_pcb (KiCad board)
At the start: 2 copper layers, 284.7 x 94.2 mm, 142 parts, among them J1 Conn_01x09_Male, J2 Conn_01x05_Male, J3 Conn_01x09_Male, K1 KEYSW, K10 KEYSW, K11 KEYSW, K12 KEYSW, K13 KEYSW, K14 KEYSW, K15 KEYSW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

Commit message: committing for foam SVGs
Parts:
- K42: footprint Switch_Keyboard_Hotswap_Kailh_mine:SW_Hotswap_Kailh_Choc_V2_ISOEnter_Gateron_LP_Stabs -> Switch_Keyboard_Hotswap_Kailh_mine:SW_Hotswap_Kailh_Choc_V2_ISOEnter_West_Gateron_LP_Stabs
