File: 2choc2flat-extmcu-iso/2choc2flat-extmcu-iso.kicad_pcb (KiCad board)
At the start: 2 copper layers, 284.7 x 94.2 mm, 142 parts, among them J1 Conn_01x09_Male, J2 Conn_01x05_Male, J3 Conn_01x09_Male, K1 KEYSW, K10 KEYSW, K11 KEYSW, K12 KEYSW, K13 KEYSW, K14 KEYSW, K15 KEYSW, K16 KEYSW, K17 KEYSW, K18 KEYSW, K19 KEYSW, K2 KEYSW, K20 KEYSW, K21 KEYSW, K22 KEYSW, K23 KEYSW, K24 KEYSW, K25 KEYSW, K26 KEYSW, K27 KEYSW, K28 KEYSW, K29 KEYSW, K29-1 KEYSW, K3 KEYSW, K30 KEYSW, K31 KEYSW, K32 KEYSW, K33 KEYSW, K34 KEYSW, K35 KEYSW, K36 KEYSW, K37 KEYSW, K38 KEYSW, K39 KEYSW, K4 KEYSW, K40 KEYSW, K41 KEYSW, K42 KEYSW, K43 KEYSW, K44 KEYSW, K45 KEYSW, K46 KEYSW, K47 KEYSW, K48 KEYSW, K49 KEYSW, K5 KEYSW, K50 KEYSW, K51 KEYSW, K52 KEYSW, K53 KEYSW, K54 KEYSW, K55 KEYSW, K56 KEYSW, K57 KEYSW, K58 KEYSW, K59 KEYSW, K6 KEYSW, K60 KEYSW, K61 KEYSW, K62 KEYSW, K63 KEYSW, K64 KEYSW, K65 KEYSW, K7 KEYSW, K8 KEYSW, K9 KEYSW

Commit message: add second caps led, minor tweaks
Parts:
- added LD2: LED, LED_SMD:LED_1206_3216Metric_ReverseMount_Hole1.8x2.4mm, B.Cu at (18.5, 53.6)
- added R2: 330R, Resistor_SMD:R_0603_1608Metric, B.Cu at (24.6, 55.1)
- R1: value R_Small_US -> 330R
Routing:
- net col14: track 39.8 -> 50.1 mm
- net Net-(D29-Pad2): track 39.7 -> 34.4 mm
- net Net-(R2-Pad2): track 0.00 -> 5.28 mm
- net col0: track 118.0 -> 120.1 mm
- net GND: vias 0 -> 1

Commit message: whoops wip
Parts:
- K42: footprint Switch_Keyboard_Hotswap_Kailh_mine:SW_Hotswap_Kailh_Choc_V2_ISOEnter_Gateron_LP_Stabs -> Switch_Keyboard_Hotswap_Kailh_mine:SW_Hotswap_Kailh_Choc_V2_ISOEnter_West_Gateron_LP_Stabs
- moved D2 8.38 mm to (28.7, 5.33), turned to 180 degrees
- moved D1 6.71 mm to (14.7, 9.65), turned to 90 degrees
- turned K1 to 180 degrees
- turned K2 to 180 degrees
- turned K65 to 0 degrees
Routing:
- net Net-(D65-Pad2): track 4.25 -> 24.4 mm
- net col1: track 100.6 -> 83.5 mm
- net col0: track 120.1 -> 107.0 mm
- net col13: track 373.0 -> 363.2 mm
- net Net-(D1-Pad2): track 11.0 -> 20.1 mm
- net row0: track 332.8 -> 324.3 mm, vias 13 -> 12
- net Net-(D2-Pad2): track 10.9 -> 11.8 mm
Other:
- board size 284.7 x 94.2 mm -> 286.7 x 94.2 mm

Commit message: version 1.4 with foam layers on eco1 and eco2
Parts:
- LD1, LD2: footprint LED_SMD:LED_1206_3216Metric_ReverseMount_Hole1.8x2.4mm -> schizobovine:LED_1206_3216Metric_ReverseMount_Hole1.8x2.4mm
- R1, R2: footprint Resistor_SMD:R_0603_1608Metric -> schizobovine:R_0603_1608Metric
- S1, S2, S6: footprint footprints:5.5_5x2.5mm -> schizobovine:3_5x2.5mm
- S3: footprint MountingHole:MountingHole_2.2mm_M2_Pad_TopOnly -> schizobovine:MountingHole_2.2mm_M2_Pad_TopOnly
- S4, S5: footprint footprints:10x5_7x2.5mm -> schizobovine:8x3.5_7x2.5mm
- moved D56 14.0 mm to (276.4, 70.9)
- moved D65 13.7 mm to (276.1, 89.9)
- moved D2 8.38 mm to (28.7, 13.7), turned to 0 degrees
- moved S5 0.23 mm to (284.0, 57.1)
- turned K15 to 0 degrees
- turned K2 to 0 degrees
- turned K56 to 0 degrees
Routing:
- net col1: track 83.5 -> 102.2 mm
- net Net-(D15-Pad2): track 4.44 -> 22.8 mm, vias 0 -> 2
- net row3: track 309.8 -> 324.7 mm, vias 9 -> 10
- net row4: track 312.8 -> 326.5 mm
- net Net-(D65-Pad2): track 24.4 -> 11.0 mm
- net col13: track 363.2 -> 352.9 mm
- net Net-(D56-Pad2): track 4.25 -> 10.9 mm
- net row0: track 324.3 -> 319.7 mm, vias 12 -> 13
- net Net-(D2-Pad2): track 11.8 -> 10.9 mm
Other:
- board text added: "2choc2flat ISO(ish) v1.4 by schizobovine <sean@yak.net>"
- board text removed: "2choc2flat ISO(ish) v1.3 by schizobovine <sean@yak.net>"
