File: 2choc2flat-extmcu-ansi-rgb/2choc2flat-extmcu-ansi-rgb.kicad_sch (KiCad schematic)
At the start: 140 parts, among them K1 KEYSW, K10 KEYSW, K11 KEYSW, K12 KEYSW, K13 KEYSW, K14 KEYSW, K16 KEYSW, K17 KEYSW, K18 KEYSW, K19 KEYSW, K2 KEYSW, K20 KEYSW, K21 KEYSW, K22 KEYSW, K23 KEYSW, K24 KEYSW, K25 KEYSW, K26 KEYSW, K27 KEYSW, K28 KEYSW, K29 KEYSW, K3 KEYSW, K31 KEYSW, K31-1 KEYSW, K32 KEYSW, K33 KEYSW, K34 KEYSW, K35 KEYSW, K36 KEYSW, K37 KEYSW, K38 KEYSW, K39 KEYSW, K4 KEYSW, K40 KEYSW, K41 KEYSW, K42 KEYSW, K44 KEYSW, K46 KEYSW, K47 KEYSW, K48 KEYSW, K49 KEYSW, K5 KEYSW, K50 KEYSW, K51 KEYSW, K52 KEYSW, K53 KEYSW, K54 KEYSW, K55 KEYSW, K56 KEYSW, K57 KEYSW, K58 KEYSW, K59 KEYSW, K6 KEYSW, K61 KEYSW, K62 KEYSW, K63 KEYSW, K67 KEYSW, K7 KEYSW, K71 KEYSW, K72 KEYSW, K73 KEYSW, K74 KEYSW, K75 KEYSW, K8 KEYSW, K9 KEYSW, U1 WS-RP2040-Tiny

Commit message: ISOish solderable version with the 3rd pin anchor
Parts:
- removed LD1, LD2: LED, schizobovine:LED_1206_3216Metric_ReverseMount_Hole1.8x2.4mm, symbol Device:LED
- removed R1, R2: 330R, Resistor_SMD:R_0603_1608Metric, symbol Device:R_Small_US
Other:
- moved on the sheet: D1, D10, D11, D12, D13, D14, D16, D17, D18, D19, D2, D20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
