File: 2choc2flat-extmcu-iso-solder/2choc2flat-extmcu-iso-solder.kicad_sch (KiCad schematic)
At the start: 139 parts, among them K1 KEYSW, K10 KEYSW, K11 KEYSW, K12 KEYSW, K13 KEYSW, K14 KEYSW, K15 KEYSW, K16 KEYSW, K17 KEYSW, K18 KEYSW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

Commit message: solderable version
Parts:
- U1: footprint schizobovine:WAVESHARE_RP2040_TINY -> schizobovine:WAVESHARE_RP2040_TINY_SLIM
