File: 2choc2flat-extmcu-iso-solder/2choc2flat-extmcu-iso-solder.kicad_pcb (KiCad board)
At the start: 2 copper layers, 286.7 x 94.2 mm, 139 parts, among them K1 KEYSW, K10 KEYSW, K11 KEYSW, K12 KEYSW, K13 KEYSW, K14 KEYSW, K15 KEYSW, K16 KEYSW, K17 KEYSW, K18 KEYSW, K19 KEYSW, K2 KEYSW, K20 KEYSW, K21 KEYSW, K22 KEYSW, K23 KEYSW, K24 KEYSW, K25 KEYSW, K26 KEYSW, K27 KEYSW, K28 KEYSW, K29 KEYSW, K3 KEYSW, K30 KEYSW, K31 KEYSW, K32 KEYSW, K33 KEYSW, K34 KEYSW, K35 KEYSW, K36 KEYSW, K37 KEYSW, K38 KEYSW, K39 KEYSW, K4 KEYSW, K40 KEYSW, K41 KEYSW, K42 KEYSW, K43 KEYSW, K44 KEYSW, K45 KEYSW, K46 KEYSW, K47 KEYSW, K48 KEYSW, K49 KEYSW, K5 KEYSW, K50 KEYSW, K51 KEYSW, K52 KEYSW, K53 KEYSW, K54 KEYSW, K55 KEYSW, K56 KEYSW, K57 KEYSW, K58 KEYSW, K59 KEYSW, K6 KEYSW, K60 KEYSW, K61 KEYSW, K62 KEYSW, K63 KEYSW, K64 KEYSW, K65 KEYSW, K7 KEYSW, K8 KEYSW, K9 KEYSW, U1 WS-RP2040-Tiny

Commit message: solderable version
Parts:
- moved D57 3.31 mm to (7.60, 79.8), turned to 0 degrees
- moved D58 1.36 mm to (28.4, 79.8), turned to 0 degrees
Routing:
- net Net-(D57-A): track 7.37 -> 3.06 mm
- net col1: track 155.9 -> 158.6 mm
- net col0: track 177.3 -> 179.8 mm
- net row4: track 287.7 -> 289.9 mm
- net Net-(D58-A): track 7.32 -> 6.04 mm
