File: 2choc2flat-extmcu-iso-rgb/2choc2flat-extmcu-iso-rgb.kicad_sch (KiCad schematic)
At the start: 220 parts, among them K1 KEYSW, K10 KEYSW, K11 KEYSW, K12 KEYSW, K13 KEYSW, K14 KEYSW, K15 KEYSW, K16 KEYSW, K17 KEYSW, K18 KEYSW, K19 KEYSW, K2 KEYSW, K20 KEYSW, K21 KEYSW, K22 KEYSW, K23 KEYSW, K24 KEYSW, K25 KEYSW, K26 KEYSW, K27 KEYSW, K28 KEYSW, K29 KEYSW, K3 KEYSW, K30 KEYSW, K31 KEYSW, K32 KEYSW, K33 KEYSW, K34 KEYSW, K35 KEYSW, K36 KEYSW, K37 KEYSW, K38 KEYSW, K39 KEYSW, K4 KEYSW, K40 KEYSW, K41 KEYSW, K42 KEYSW, K43 KEYSW, K44 KEYSW, K45 KEYSW, K46 KEYSW, K47 KEYSW, K48 KEYSW, K49 KEYSW, K5 KEYSW, K50 KEYSW, K51 KEYSW, K52 KEYSW, K53 KEYSW, K54 KEYSW, K55 KEYSW, K56 KEYSW, K57 KEYSW, K58 KEYSW, K59 KEYSW, K6 KEYSW, K60 KEYSW, K61 KEYSW, K62 KEYSW, K63 KEYSW, K64 KEYSW, K65 KEYSW, K7 KEYSW, K8 KEYSW, K9 KEYSW, U1 WS-RP2040-Tiny, U2 74LVC2G125

Commit message: redo underglow because i failed to map the pads correctly
Parts:
- BD1, BD10, BD11, BD12, BD13, BD14, BD15, BD16, BD2, BD3, BD4, BD5, BD6, BD7, BD8, BD9: symbol LED:WS2812B -> schizobovine:WS2812B
- K60: footprint Switch_Keyboard_Hotswap_Kailh_mine:SW_Hotswap_Kailh_Choc_V2_6.25u_special -> Switch_Keyboard_Hotswap_Kailh_mine:SW_Hotswap_Kailh_Choc_V2_6.25u_special2
Connections:
- net +5V: now also BD1.4 (VDD), BD10.4 (VDD), BD11.4 (VDD), BD12.4 (VDD), BD13.4 (VDD), BD14.4 (VDD), BD15.4 (VDD), BD16.4 (VDD), BD2.4 (VDD), BD3.4 (VDD), BD4.4 (VDD), BD5.4 (VDD), BD6.4 (VDD), BD7.4 (VDD), BD8.4 (VDD), BD9.4 (VDD); no longer BD1.1 (VDD), BD10.1 (VDD), BD11.1 (VDD), BD12.1 (VDD), BD13.1 (VDD), BD14.1 (VDD), BD15.1 (VDD), BD16.1 (VDD), BD2.1 (VDD), BD3.1 (VDD), BD4.1 (VDD), BD5.1 (VDD), BD6.1 (VDD), BD7.1 (VDD), BD8.1 (VDD), BD9.1 (VDD)
- net GND: now also BD1.2 (VSS), BD10.2 (VSS), BD11.2 (VSS), BD12.2 (VSS), BD13.2 (VSS), BD14.2 (VSS), BD15.2 (VSS), BD16.2 (VSS), BD2.2 (VSS), BD3.2 (VSS), BD4.2 (VSS), BD5.2 (VSS), BD6.2 (VSS), BD7.2 (VSS), BD8.2 (VSS), BD9.2 (VSS); no longer BD1.3 (VSS), BD10.3 (VSS), BD11.3 (VSS), BD12.3 (VSS), BD13.3 (VSS), BD14.3 (VSS), BD15.3 (VSS), BD16.3 (VSS), BD2.3 (VSS), BD3.3 (VSS), BD4.3 (VSS), BD5.3 (VSS), BD6.3 (VSS), BD7.3 (VSS), BD8.3 (VSS), BD9.3 (VSS)
- net underglow_5v: now also BD1.3 (DIN); no longer BD1.4 (DIN)
- new net: BD2.1 (DOUT), BD3.3 (DIN)
- new net: BD1.1 (DOUT), BD2.3 (DIN)
- new net: BD11.1 (DOUT), BD12.3 (DIN)
- new net: BD10.1 (DOUT), BD11.3 (DIN)
- new net: BD15.1 (DOUT), BD16.3 (DIN)
- new net: BD10.3 (DIN), BD9.1 (DOUT)
- new net: BD8.1 (DOUT), BD9.3 (DIN)
- new net: BD5.1 (DOUT), BD6.3 (DIN)
- new net: BD4.1 (DOUT), BD5.3 (DIN)
- new net: BD13.1 (DOUT), BD14.3 (DIN)
- new net: BD12.1 (DOUT), BD13.3 (DIN)
- new net: BD14.1 (DOUT), BD15.3 (DIN)
- new net: BD6.1 (DOUT), BD7.3 (DIN)
- new net: BD3.1 (DOUT), BD4.3 (DIN)
- new net: BD7.1 (DOUT), BD8.3 (DIN)

Commit message: fixing more fuckups
Connections:
- net +5V: now also LD1.1 (VDD), LD10.1 (VDD), LD11.1 (VDD), LD12.1 (VDD), LD13.1 (VDD), LD14.1 (VDD), LD15.1 (VDD), LD16.1 (VDD), LD17.1 (VDD), LD18.1 (VDD), LD19.1 (VDD), LD2.1 (VDD), LD20.1 (VDD), LD21.1 (VDD), LD22.1 (VDD), LD23.1 (VDD), LD24.1 (VDD), LD25.1 (VDD), LD26.1 (VDD), LD27.1 (VDD), LD28.1 (VDD), LD29.1 (VDD), LD3.1 (VDD), LD30.1 (VDD), LD31.1 (VDD), LD32.1 (VDD), LD33.1 (VDD), LD34.1 (VDD), LD35.1 (VDD), LD36.1 (VDD), LD37.1 (VDD), LD38.1 (VDD), LD39.1 (VDD), LD4.1 (VDD), LD40.1 (VDD), LD41.1 (VDD), LD42.1 (VDD), LD43.1 (VDD), LD44.1 (VDD), LD45.1 (VDD), LD46.1 (VDD), LD47.1 (VDD), LD48.1 (VDD), LD49.1 (VDD), LD5.1 (VDD), LD50.1 (VDD), LD51.1 (VDD), LD52.1 (VDD), LD53.1 (VDD), LD54.1 (VDD), LD55.1 (VDD), LD56.1 (VDD), LD57.1 (VDD), LD58.1 (VDD), LD59.1 (VDD), LD6.1 (VDD), LD60.1 (VDD), LD61.1 (VDD), LD62.1 (VDD), LD63.1 (VDD), LD64.1 (VDD), LD65.1 (VDD), LD7.1 (VDD), LD8.1 (VDD), LD9.1 (VDD); no longer LD1.4 (VDD), LD10.4 (VDD), LD11.4 (VDD), LD12.4 (VDD), LD13.4 (VDD), LD14.4 (VDD), LD15.4 (VDD), LD16.4 (VDD), LD17.4 (VDD), LD18.4 (VDD), LD19.4 (VDD), LD2.4 (VDD), LD20.4 (VDD), LD21.4 (VDD), LD22.4 (VDD), LD23.4 (VDD), LD24.4 (VDD), LD25.4 (VDD), LD26.4 (VDD), LD27.4 (VDD), LD28.4 (VDD), LD29.4 (VDD), LD3.4 (VDD), LD30.4 (VDD), LD31.4 (VDD), LD32.4 (VDD), LD33.4 (VDD), LD34.4 (VDD), LD35.4 (VDD), LD36.4 (VDD), LD37.4 (VDD), LD38.4 (VDD), LD39.4 (VDD), LD4.4 (VDD), LD40.4 (VDD), LD41.4 (VDD), LD42.4 (VDD), LD43.4 (VDD), LD44.4 (VDD), LD45.4 (VDD), LD46.4 (VDD), LD47.4 (VDD), LD48.4 (VDD), LD49.4 (VDD), LD5.4 (VDD), LD50.4 (VDD), LD51.4 (VDD), LD52.4 (VDD), LD53.4 (VDD), LD54.4 (VDD), LD55.4 (VDD), LD56.4 (VDD), LD57.4 (VDD), LD58.4 (VDD), LD59.4 (VDD), LD6.4 (VDD), LD60.4 (VDD), LD61.4 (VDD), LD62.4 (VDD), LD63.4 (VDD), LD64.4 (VDD), LD65.4 (VDD), LD7.4 (VDD), LD8.4 (VDD), LD9.4 (VDD)
- net GND: now also LD1.3 (VSS), LD10.3 (VSS), LD11.3 (VSS), LD12.3 (VSS), LD13.3 (VSS), LD14.3 (VSS), LD15.3 (VSS), LD16.3 (VSS), LD17.3 (VSS), LD18.3 (VSS), LD19.3 (VSS), LD2.3 (VSS), LD20.3 (VSS), LD21.3 (VSS), LD22.3 (VSS), LD23.3 (VSS), LD24.3 (VSS), LD25.3 (VSS), LD26.3 (VSS), LD27.3 (VSS), LD28.3 (VSS), LD29.3 (VSS), LD3.3 (VSS), LD30.3 (VSS), LD31.3 (VSS), LD32.3 (VSS), LD33.3 (VSS), LD34.3 (VSS), LD35.3 (VSS), LD36.3 (VSS), LD37.3 (VSS), LD38.3 (VSS), LD39.3 (VSS), LD4.3 (VSS), LD40.3 (VSS), LD41.3 (VSS), LD42.3 (VSS), LD43.3 (VSS), LD44.3 (VSS), LD45.3 (VSS), LD46.3 (VSS), LD47.3 (VSS), LD48.3 (VSS), LD49.3 (VSS), LD5.3 (VSS), LD50.3 (VSS), LD51.3 (VSS), LD52.3 (VSS), LD53.3 (VSS), LD54.3 (VSS), LD55.3 (VSS), LD56.3 (VSS), LD57.3 (VSS), LD58.3 (VSS), LD59.3 (VSS), LD6.3 (VSS), LD60.3 (VSS), LD61.3 (VSS), LD62.3 (VSS), LD63.3 (VSS), LD64.3 (VSS), LD65.3 (VSS), LD7.3 (VSS), LD8.3 (VSS), LD9.3 (VSS); no longer LD1.2 (VSS), LD10.2 (VSS), LD11.2 (VSS), LD12.2 (VSS), LD13.2 (VSS), LD14.2 (VSS), LD15.2 (VSS), LD16.2 (VSS), LD17.2 (VSS), LD18.2 (VSS), LD19.2 (VSS), LD2.2 (VSS), LD20.2 (VSS), LD21.2 (VSS), LD22.2 (VSS), LD23.2 (VSS), LD24.2 (VSS), LD25.2 (VSS), LD26.2 (VSS), LD27.2 (VSS), LD28.2 (VSS), LD29.2 (VSS), LD3.2 (VSS), LD30.2 (VSS), LD31.2 (VSS), LD32.2 (VSS), LD33.2 (VSS), LD34.2 (VSS), LD35.2 (VSS), LD36.2 (VSS), LD37.2 (VSS), LD38.2 (VSS), LD39.2 (VSS), LD4.2 (VSS), LD40.2 (VSS), LD41.2 (VSS), LD42.2 (VSS), LD43.2 (VSS), LD44.2 (VSS), LD45.2 (VSS), LD46.2 (VSS), LD47.2 (VSS), LD48.2 (VSS), LD49.2 (VSS), LD5.2 (VSS), LD50.2 (VSS), LD51.2 (VSS), LD52.2 (VSS), LD53.2 (VSS), LD54.2 (VSS), LD55.2 (VSS), LD56.2 (VSS), LD57.2 (VSS), LD58.2 (VSS), LD59.2 (VSS), LD6.2 (VSS), LD60.2 (VSS), LD61.2 (VSS), LD62.2 (VSS), LD63.2 (VSS), LD64.2 (VSS), LD65.2 (VSS), LD7.2 (VSS), LD8.2 (VSS), LD9.2 (VSS)
- net per_key_rgb_5v: now also LD1.4 (DIN); no longer LD1.3 (DIN)
- new net: LD34.2 (DOUT), LD35.4 (DIN)
- new net: LD33.2 (DOUT), LD34.4 (DIN)
- new net: LD12.2 (DOUT), LD13.4 (DIN)
- new net: LD11.2 (DOUT), LD12.4 (DIN)
- new net: LD6.2 (DOUT), LD7.4 (DIN)
- new net: LD5.2 (DOUT), LD6.4 (DIN)
- new net: LD36.2 (DOUT), LD37.4 (DIN)
- new net: LD35.2 (DOUT), LD36.4 (DIN)
- new net: LD3.2 (DOUT), LD4.4 (DIN)
- new net: LD2.2 (DOUT), LD3.4 (DIN)
- new net: LD62.2 (DOUT), LD63.4 (DIN)
- new net: LD61.2 (DOUT), LD62.4 (DIN)
- new net: LD59.2 (DOUT), LD60.4 (DIN)
- new net: LD58.2 (DOUT), LD59.4 (DIN)
- new net: LD40.2 (DOUT), LD41.4 (DIN)
- new net: LD39.2 (DOUT), LD40.4 (DIN)
- new net: LD4.2 (DOUT), LD5.4 (DIN)
- new net: LD27.4 (DIN), LD28.2 (DOUT)
- new net: LD15.2 (DOUT), LD28.4 (DIN)
- new net: LD55.4 (DIN), LD56.2 (DOUT)
- new net: LD42.2 (DOUT), LD56.4 (DIN)
- new net: LD53.4 (DIN), LD54.2 (DOUT)
- new net: LD54.4 (DIN), LD55.2 (DOUT)
- new net: LD37.2 (DOUT), LD38.4 (DIN)
- new net: LD25.4 (DIN), LD26.2 (DOUT)
- new net: LD26.4 (DIN), LD27.2 (DOUT)
- new net: LD20.4 (DIN), LD21.2 (DOUT)
- new net: LD21.4 (DIN), LD22.2 (DOUT)
- new net: LD45.4 (DIN), LD46.2 (DOUT)
- new net: LD46.4 (DIN), LD47.2 (DOUT)
- new net: LD18.4 (DIN), LD19.2 (DOUT)
- new net: LD19.4 (DIN), LD20.2 (DOUT)
- new net: LD1.2 (DOUT), LD2.4 (DIN)
- new net: LD22.4 (DIN), LD23.2 (DOUT)
- new net: LD23.4 (DIN), LD24.2 (DOUT)
- new net: LD7.2 (DOUT), LD8.4 (DIN)
- new net: LD17.4 (DIN), LD18.2 (DOUT)
- new net: LD31.2 (DOUT), LD32.4 (DIN)
- new net: LD30.2 (DOUT), LD31.4 (DIN)
- new net: LD64.2 (DOUT), LD65.4 (DIN)
- new net: LD63.2 (DOUT), LD64.4 (DIN)
- new net: LD13.2 (DOUT), LD14.4 (DIN)
- new net: LD47.4 (DIN), LD48.2 (DOUT)
- new net: LD24.4 (DIN), LD25.2 (DOUT)
- new net: LD51.4 (DIN), LD52.2 (DOUT)
- new net: LD52.4 (DIN), LD53.2 (DOUT)
- new net: LD48.4 (DIN), LD49.2 (DOUT)
- new net: LD8.2 (DOUT), LD9.4 (DIN)
- new net: LD29.2 (DOUT), LD30.4 (DIN)
- new net: LD57.2 (DOUT), LD58.4 (DIN)
- new net: LD43.4 (DIN), LD44.2 (DOUT)
- new net: LD44.4 (DIN), LD45.2 (DOUT)
- new net: LD10.2 (DOUT), LD11.4 (DIN)
- new net: LD10.4 (DIN), LD9.2 (DOUT)
- new net: LD16.4 (DIN), LD17.2 (DOUT)
- new net: LD50.4 (DIN), LD51.2 (DOUT)
- new net: LD60.2 (DOUT), LD61.4 (DIN)
- new net: LD43.2 (DOUT), LD57.4 (DIN)
- new net: LD41.2 (DOUT), LD42.4 (DIN)
- new net: LD16.2 (DOUT), LD29.4 (DIN)
- new net: LD49.4 (DIN), LD50.2 (DOUT)
- new net: LD38.2 (DOUT), LD39.4 (DIN)
- new net: LD32.2 (DOUT), LD33.4 (DIN)
- new net: LD14.2 (DOUT), LD15.4 (DIN)
Changed lines of the file:
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@@
     )
   )
-  (symbol (lib_id "power:+5V") (at 28.575 164.465 0) (mirror y) (unit 1)
+  (symbol (lib_name "+5V_5") (lib_id "power:+5V") (at 28.575 164.465 0) (mirror y) (unit 1)
     (in_bom yes) (on_board yes) (dnp no) (fields_autoplaced)
     (property "Reference" "#PWR0106" (at 28.575 168.275 0)
@@
     )
   )
-  (symbol (lib_id "power:+5V") (at 57.15 253.365 0) (mirror y) (unit 1)
+  (symbol (lib_name "+5V_3") (lib_id "power:+5V") (at 57.15 253.365 0) (mirror y) (unit 1)
     (in_bom yes) (on_board yes) (dnp no) (fields_autoplaced)
     (property "Reference" "#PWR0109" (at 57.15 257.175 0)
@@
     )
   )
-  (symbol (lib_id "power:+5V") (at 41.91 209.55 0) (mirror y) (unit 1)
+  (symbol (lib_name "+5V_2") (lib_id "power:+5V") (at 41.91 209.55 0) (mirror y) (unit 1)
     (in_bom yes) (on_board yes) (dnp no) (fields_autoplaced)
     (property "Reference" "#PWR0113" (at 41.91 213.36 0)
@@
     )
   )
-  (symbol (lib_id "power:+5V") (at 35.56 187.325 0) (mirror y) (unit 1)
+  (symbol (lib_name "+5V_4") (lib_id "power:+5V") (at 35.56 187.325 0) (mirror y) (unit 1)
     (in_bom yes) (on_board yes) (dnp no) (fields_autoplaced)
     (property "Reference" "#PWR0120" (at 35.56 191.135 0)
@@
     )
   )
-  (symbol (lib_id "power:+5V") (at 49.53 231.775 0) (mirror y) (unit 1)
+  (symbol (lib_name "+5V_1") (lib_id "power:+5V") (at 49.53 231.775 0) (mirror y) (unit 1)
     (in_bom yes) (on_board yes) (dnp no) (fields_autoplaced)
     (property "Reference" "#PWR0112" (at 49.53 235.585 0)
